Commit message: Isaacsim support.

File: xarm_description/urdf/lite6/lite6.ros2_control.xacro (robot description, xacro)
@@ -12,5 +12,6 @@
     joint5_lower_limit:=${-2.1642}  joint5_upper_limit:=${2.1642}
     joint6_lower_limit:=${-2.0*pi}  joint6_upper_limit:=${2.0*pi}">
-    <ros2_control name="${prefix}${ros2_control_plugin}" type="system">
+    <!-- FIXME There is bug with this name -->
+    <ros2_control name="${prefix}isaacsim" type="system">
       <hardware>
         <plugin>${ros2_control_plugin}</plugin>
@@ -26,4 +27,8 @@
           <param name="robot_type">lite</param>
           <param name="add_gripper">${add_gripper}</param>
+        </xacro:if>
+        <xacro:if value="${ros2_control_plugin == 'topic_based_ros2_control/TopicBasedSystem'}">
+          <param name="joint_commands_topic">/isaac/joint_command</param>
+          <param name="joint_states_topic">/isaac/joint_states</param>
         </xacro:if>
       </hardware>
@@ -106,4 +111,18 @@
         <!-- <state_interface name="effort"/> -->
       </joint>
+      <!-- Having fingers under same ros2_control to have one message on /isaac/joint_command -->
+      <xacro:if value="${ros2_control_plugin == 'topic_based_ros2_control/TopicBasedSystem'}">
+        <joint name="${prefix}finger_joint1">
+          <command_interface name="position">
+          </command_interface>
+          <command_interface name="velocity">
+            <param name="min">-3.14</param>
+            <param name="max">3.14</param>
+          </command_interface>
+          <state_interface name="position"/>
+          <state_interface name="velocity"/>
+          <!-- <state_interface name="effort"/> -->
+        </joint>
+      </xacro:if>
     </ros2_control>
   </xacro:macro>
